File: hardware/Tempatroller.brd (EAGLE design)
At the start: 91.4 x 53.3 mm, 34 parts, among them U1 VSK-S5, U2 MAX31856, U3 LTV-354T, U4 FODM3053, U5 T25

Commit message: Packed all parts into local project library. Renamed project files.
Parts:
- AC/L, AC/N, HTR/L, HTR/N: device ReflowOvenController:QUICK-1 -> Tempatroller:QUICK-1
- AIO: device ReflowOvenController:1X06 -> Tempatroller:1X06
- C1: device ReflowOvenController:153CLV-1014 -> Tempatroller:153CLV-1014
- C2, C3, C4, C5, C6, C7: device ReflowOvenController:C0805 -> Tempatroller:C0805
- DIO-H: device ReflowOvenController:1X10 -> Tempatroller:1X10
- DIO-L, POWER: device ReflowOvenController:1X08 -> Tempatroller:1X08
- F1: device ReflowOvenController:2SMD-2410 -> Tempatroller:2SMD-2410
- JP1, JP3: device SmslsTron:SCREWTERMINAL-5MM-2 -> Tempatroller:SCREWTERMINAL-5MM-2
- LED1, LED2, LED3: device SmslsTron:CHIP-LED0805 -> Tempatroller:CHIP-LED0805
- R1, R2, R4: device ReflowOvenController:R1206 -> Tempatroller:R1206
- R3: device ReflowOvenController:R0805 -> Tempatroller:R0805
- R5, R6, R7: device SmslsTron:R0805 -> Tempatroller:R0805
- U$1: device SmslsTron:SILK_QC -> Tempatroller:SILK_QC
- U1: device ReflowOvenController:VSK-S5 -> Tempatroller:VSK-S5
- U2: device ReflowOvenController:TSSOP14 -> Tempatroller:TSSOP14
- U3, U4: device ReflowOvenController:SOP-4 -> Tempatroller:SOP-4
- U5: device ReflowOvenController:TO263-3 -> Tempatroller:TO263-3
