File: hardware/Tempatroller.sch (EAGLE design)
At the start: 34 parts, among them U1 VSK-S5, U2 MAX31856, U3 LTV-354T, U4 FODM3053, U5 T25

Commit message: Packed all parts into local project library. Renamed project files.
Parts:
- AC/L, AC/N, HTR/L, HTR/N: device ReflowOvenController:JMP-1-QUICK -> Tempatroller:JMP-1-QUICK
- AIO: device ReflowOvenController:PINHD-1X6TH -> Tempatroller:PINHD-1X6TH
- C1: device ReflowOvenController:CPOL-US153CLV-1014 -> Tempatroller:CPOL-US153CLV-1014
- C2, C3, C4, C5, C6, C7: device ReflowOvenController:C-USC0805 -> Tempatroller:C-USC0805
- DIO-H: device ReflowOvenController:PINHD-1X10TH -> Tempatroller:PINHD-1X10TH
- DIO-L, POWER: device ReflowOvenController:PINHD-1X8TH -> Tempatroller:PINHD-1X8TH
- F1: device ReflowOvenController:FUSE2410 -> Tempatroller:FUSE2410
- JP1, JP3: device SmslsTron:M025MM -> Tempatroller:M025MM
- LED1, LED2, LED3: device SmslsTron:LEDCHIP-LED0805 -> Tempatroller:LEDCHIP-LED0805
- R1, R2, R4: device ReflowOvenController:R-US_R1206 -> Tempatroller:R-US_R1206
- R3: device ReflowOvenController:R-US_R0805 -> Tempatroller:R-US_R0805
- R5, R6, R7: device SmslsTron:R-US_R0805 -> Tempatroller:R-US_R0805
- U$1: device SmslsTron:SILK_QC -> Tempatroller:SILK_QC
- U1: device ReflowOvenController:VSK-S5 -> Tempatroller:VSK-S5
- U2: device ReflowOvenController:MAX31856 -> Tempatroller:MAX31856
- U3: device ReflowOvenController:LTV-354T -> Tempatroller:LTV-354T
- U4: device ReflowOvenController:FODM3053 -> Tempatroller:FODM3053
- U5: device ReflowOvenController:T835-TO263 -> Tempatroller:T835-TO263
Changed lines of the file:
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@@
 </classes>
 <parts>
-<part name="DIO-L" library="ReflowOvenController" deviceset="PINHD-1X8" device="TH" value="8x1F-H8.5"/>
-<part name="DIO-H" library="ReflowOvenController" deviceset="PINHD-1X10" device="TH" value="10x1F-H8.5"/>
-<part name="AIO" library="ReflowOvenController" deviceset="PINHD-1X6" device="TH" value="6x1F-H8.5"/>
-<part name="U1" library="ReflowOvenController" deviceset="VSK-S5" device="">
+<part name="DIO-L" library="Tempatroller" deviceset="PINHD-1X8" device="TH" value="8x1F-H8.5"/>
+<part name="DIO-H" library="Tempatroller" deviceset="PINHD-1X10" device="TH" value="10x1F-H8.5"/>
+<part name="AIO" library="Tempatroller" deviceset="PINHD-1X6" device="TH" value="6x1F-H8.5"/>
+<part name="U1" library="Tempatroller" deviceset="VSK-S5" device="">
 <attribute name="PN-DK" value="102-2387-ND"/>
 </part>
-<part name="POWER" library="ReflowOvenController" deviceset="PINHD-1X8" device="TH" value="8x1F-H8.5"/>
-<part name="C1" library="ReflowOvenController" deviceset="CPOL-US" device="153CLV-1014" value="220u">
+<part name="POWER" library="Tempatroller" deviceset="PINHD-1X8" device="TH" value="8x1F-H8.5"/>
+<part name="C1" library="Tempatroller" deviceset="CPOL-US" device="153CLV-1014" value="220u">
 <attribute name="PN-DK" value="PCE3812CT-ND"/>
 </part>
-<part name="C2" library="ReflowOvenController" deviceset="C-US" device="C0805" value="1u"/>
-<part name="U2" library="ReflowOvenController" deviceset="MAX31856" device=""/>
-<part name="C3" library="ReflowOvenController" deviceset="C-US" device="C0805" value="100n"/>
-<part name="C4" library="ReflowOvenController" deviceset="C-US" device="C0805" value="100n"/>
-<part name="C5" library="ReflowOvenController" deviceset="C-US" device="C0805" value="100n"/>
-<part name="C6" library="ReflowOvenController" deviceset="C-US" device="C0805" value="10n"/>
-<part name="C7" library="ReflowOvenController" deviceset="C-US" device="C0805" value="10n"/>
-<part name="U3" library="ReflowOvenController" deviceset="LTV-354T" device=""/>
-<part name="R1" library="ReflowOvenController" deviceset="R-US_" device="R1206" value="47k"/>
-<part name="R2" library="ReflowOvenController" deviceset="R-US_" device="R1206" value="47k"/>
-<part name="F1" library="ReflowOvenController" deviceset="FUSE" device="2410" value="250V/1A">
+<part name="C2" library="Tempatroller" deviceset="C-US" device="C0805" value="1u"/>
+<part name="U2" library="Tempatroller" deviceset="MAX31856" device=""/>
+<part name="C3" library="Tempatroller" deviceset="C-US" device="C0805" value="100n"/>
+<part name="C4" library="Tempatroller" deviceset="C-US" device="C0805" value="100n"/>
+<part name="C5" library="Tempatroller" deviceset="C-US" device="C0805" value="100n"/>
+<part name="C6" library="Tempatroller" deviceset="C-US" device="C0805" value="10n"/>
+<part name="C7" library="Tempatroller" deviceset="C-US" device="C0805" value="10n"/>
+<part name="U3" library="Tempatroller" deviceset="LTV-354T" device=""/>
+<part name="R1" library="Tempatroller" deviceset="R-US_" device="R1206" value="47k"/>
+<part name="R2" library="Tempatroller" deviceset="R-US_" device="R1206" value="47k"/>
+<part name="F1" library="Tempatroller" deviceset="FUSE" device="2410" value="250V/1A">
 <attribute name="MPN" value="0454001.MR"/>
 <attribute name="PN-DK" value="F3144CT-ND"/>
 </part>
-<part name="AC/L" library="ReflowOvenController" deviceset="JMP-1" device="-QUICK"/>
-<part name="AC/N" library="ReflowOvenController" deviceset="JMP-1" device="-QUICK"/>
-<part name="JP1" library="SmslsTron" deviceset="M02" device="5MM" value="M025MM"/>
-<part name="JP3" library="SmslsTron" deviceset="M02" device="5MM" value="M025MM"/>
-<part name="U4" library="ReflowOvenController" deviceset="FODM3053" device=""/>
-<part name="R3" library="ReflowOvenController" deviceset="R-US_" device="R0805" value="100"/>
-<part name="HTR/L" library="ReflowOvenController" deviceset="JMP-1" device="-QUICK"/>
-<part name="HTR/N" library="ReflowOvenController" deviceset="JMP-1" device="-QUICK"/>
-<part name="U5" library="ReflowOvenController" deviceset="T835" device="-TO263" value="T25">
+<part name="AC/L" library="Tempatroller" deviceset="JMP-1" device="-QUICK"/>
+<part name="AC/N" library="Tempatroller" deviceset="JMP-1" device="-QUICK"/>
+<part name="JP1" library="Tempatroller" deviceset="M02" device="5MM" value="M025MM"/>
+<part name="JP3" library="Tempatroller" deviceset="M02" device="5MM" value="M025MM"/>
+<part name="U4" library="Tempatroller" deviceset="FODM3053" device=""/>
+<part name="R3" library="Tempatroller" deviceset="R-US_" device="R0805" value="100"/>
+<part name="HTR/L" library="Tempatroller" deviceset="JMP-1" device="-QUICK"/>
+<part name="HTR/N" library="Tempatroller" deviceset="JMP-1" device="-QUICK"/>
+<part name="U5" library="Tempatroller" deviceset="T835" device="-TO263" value="T25">
 <attribute name="PN-DK" value="497-10581-1-ND"/>
 </part>
-<part name="R4" library="ReflowOvenController" deviceset="R-US_" device="R1206" value="1k"/>
-<part name="FRAME1" library="SmslsTron" deviceset="LETTER_L" device="">
+<part name="R4" library="Tempatroller" deviceset="R-US_" device="R1206" value="1k"/>
+<part name="FRAME1" library="Tempatroller" deviceset="LETTER_L" device="">
 <attribute name="SECTION" value=""/>
 </part>
-<part name="U$1" library="SmslsTron" deviceset="SILK_QC" device="">
+<part name="U$1" library="Tempatroller" deviceset="SILK_QC" device="">
 <attribute name="PRODUCT" value="TempController"/>
 <attribute name="REV" value="1B"/>
 </part>
-<part name="R5" library="SmslsTron" deviceset="R-US_" device="R0805" value="390"/>
-<part name="LED1" library="SmslsTron" deviceset="LED" device="CHIP-LED0805">
+<part name="R5" library="Tempatroller" deviceset="R-US_" device="R0805" value="390"/>
+<part name="LED1" library="Tempatroller" deviceset="LED" device="CHIP-LED0805">
 <attribute name="LABEL" value="PWR"/>
 </part>
-<part name="R6" library="SmslsTron" deviceset="R-US_" device="R0805" value="390"/>
-<part name="LED2" library="SmslsTron" deviceset="LED" device="CHIP-LED0805">
+<part name="R6" library="Tempatroller" deviceset="R-US_" device="R0805" value="390"/>
+<part name="LED2" library="Tempatroller" deviceset="LED" device="CHIP-LED0805">
 <attribute name="LABEL" value="HB"/>
 </part>
-<part name="R7" library="SmslsTron" deviceset="R-US_" device="R0805" value="390"/>
-<part name="LED3" library="SmslsTron" deviceset="LED" device="CHIP-LED0805">
+<part name="R7" library="Tempatroller" deviceset="R-US_" device="R0805" value="390"/>
+<part name="LED3" library="Tempatroller" deviceset="LED" device="CHIP-LED0805">
 <attribute name="LABEL" value="SSR"/>
 </part>
