File: hardware/ThermoBot.sch (EAGLE design)
At the start: 34 parts, among them U1 VSK-S5, U2 MAX31856, U3 LTV-354T, U4 FODM3053, U5 T25

Commit message: Renamed to ThermoBot
Parts:
- AC/L, AC/N, HTR/L, HTR/N: device Tempatroller:JMP-1-QUICK -> ThermoBot:JMP-1-QUICK
- AIO: device Tempatroller:PINHD-1X6TH -> ThermoBot:PINHD-1X6TH
- C1: device Tempatroller:CPOL-US153CLV-1014 -> ThermoBot:CPOL-US153CLV-1014
- C2, C3, C4, C5, C6, C7: device Tempatroller:C-USC0805 -> ThermoBot:C-USC0805
- DIO-H: device Tempatroller:PINHD-1X10TH -> ThermoBot:PINHD-1X10TH
- DIO-L, POWER: device Tempatroller:PINHD-1X8TH -> ThermoBot:PINHD-1X8TH
- F1: device Tempatroller:FUSE2410 -> ThermoBot:FUSE2410
- JP1, JP3: device Tempatroller:M025MM -> ThermoBot:M025MM
- LED1, LED2, LED3: device Tempatroller:LEDCHIP-LED0805 -> ThermoBot:LEDCHIP-LED0805
- R1, R2, R4: device Tempatroller:R-US_R1206 -> ThermoBot:R-US_R1206
- R3, R5, R6, R7: device Tempatroller:R-US_R0805 -> ThermoBot:R-US_R0805
- U$1: device Tempatroller:SILK_QC -> ThermoBot:SILK_QC; PRODUCT TempController -> ThermoBot
- U1: device Tempatroller:VSK-S5 -> ThermoBot:VSK-S5
- U2: device Tempatroller:MAX31856 -> ThermoBot:MAX31856
- U3: device Tempatroller:LTV-354T -> ThermoBot:LTV-354T
- U4: device Tempatroller:FODM3053 -> ThermoBot:FODM3053
- U5: device Tempatroller:T835-TO263 -> ThermoBot:T835-TO263
Changed lines of the file:
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@@
 </classes>
 <parts>
-<part name="DIO-L" library="Tempatroller" deviceset="PINHD-1X8" device="TH" value="8x1F-H8.5"/>
-<part name="DIO-H" library="Tempatroller" deviceset="PINHD-1X10" device="TH" value="10x1F-H8.5"/>
-<part name="AIO" library="Tempatroller" deviceset="PINHD-1X6" device="TH" value="6x1F-H8.5"/>
-<part name="U1" library="Tempatroller" deviceset="VSK-S5" device="">
+<part name="DIO-L" library="ThermoBot" deviceset="PINHD-1X8" device="TH" value="8x1F-H8.5"/>
+<part name="DIO-H" library="ThermoBot" deviceset="PINHD-1X10" device="TH" value="10x1F-H8.5"/>
+<part name="AIO" library="ThermoBot" deviceset="PINHD-1X6" device="TH" value="6x1F-H8.5"/>
+<part name="U1" library="ThermoBot" deviceset="VSK-S5" device="">
 <attribute name="PN-DK" value="102-2387-ND"/>
 </part>
-<part name="POWER" library="Tempatroller" deviceset="PINHD-1X8" device="TH" value="8x1F-H8.5"/>
-<part name="C1" library="Tempatroller" deviceset="CPOL-US" device="153CLV-1014" value="220u">
+<part name="POWER" library="ThermoBot" deviceset="PINHD-1X8" device="TH" value="8x1F-H8.5"/>
+<part name="C1" library="ThermoBot" deviceset="CPOL-US" device="153CLV-1014" value="220u">
 <attribute name="PN-DK" value="PCE3812CT-ND"/>
 </part>
-<part name="C2" library="Tempatroller" deviceset="C-US" device="C0805" value="1u"/>
-<part name="U2" library="Tempatroller" deviceset="MAX31856" device=""/>
-<part name="C3" library="Tempatroller" deviceset="C-US" device="C0805" value="100n"/>
-<part name="C4" library="Tempatroller" deviceset="C-US" device="C0805" value="100n"/>
-<part name="C5" library="Tempatroller" deviceset="C-US" device="C0805" value="100n"/>
-<part name="C6" library="Tempatroller" deviceset="C-US" device="C0805" value="10n"/>
-<part name="C7" library="Tempatroller" deviceset="C-US" device="C0805" value="10n"/>
-<part name="U3" library="Tempatroller" deviceset="LTV-354T" device=""/>
-<part name="R1" library="Tempatroller" deviceset="R-US_" device="R1206" value="47k"/>
-<part name="R2" library="Tempatroller" deviceset="R-US_" device="R1206" value="47k"/>
-<part name="F1" library="Tempatroller" deviceset="FUSE" device="2410" value="250V/1A">
+<part name="C2" library="ThermoBot" deviceset="C-US" device="C0805" value="1u"/>
+<part name="U2" library="ThermoBot" deviceset="MAX31856" device=""/>
+<part name="C3" library="ThermoBot" deviceset="C-US" device="C0805" value="100n"/>
+<part name="C4" library="ThermoBot" deviceset="C-US" device="C0805" value="100n"/>
+<part name="C5" library="ThermoBot" deviceset="C-US" device="C0805" value="100n"/>
+<part name="C6" library="ThermoBot" deviceset="C-US" device="C0805" value="10n"/>
+<part name="C7" library="ThermoBot" deviceset="C-US" device="C0805" value="10n"/>
+<part name="U3" library="ThermoBot" deviceset="LTV-354T" device=""/>
+<part name="R1" library="ThermoBot" deviceset="R-US_" device="R1206" value="47k"/>
+<part name="R2" library="ThermoBot" deviceset="R-US_" device="R1206" value="47k"/>
+<part name="F1" library="ThermoBot" deviceset="FUSE" device="2410" value="250V/1A">
 <attribute name="MPN" value="0454001.MR"/>
 <attribute name="PN-DK" value="F3144CT-ND"/>
 </part>
-<part name="AC/L" library="Tempatroller" deviceset="JMP-1" device="-QUICK"/>
-<part name="AC/N" library="Tempatroller" deviceset="JMP-1" device="-QUICK"/>
-<part name="JP1" library="Tempatroller" deviceset="M02" device="5MM" value="M025MM"/>
-<part name="JP3" library="Tempatroller" deviceset="M02" device="5MM" value="M025MM"/>
-<part name="U4" library="Tempatroller" deviceset="FODM3053" device=""/>
-<part name="R3" library="Tempatroller" deviceset="R-US_" device="R0805" value="100"/>
-<part name="HTR/L" library="Tempatroller" deviceset="JMP-1" device="-QUICK"/>
-<part name="HTR/N" library="Tempatroller" deviceset="JMP-1" device="-QUICK"/>
-<part name="U5" library="Tempatroller" deviceset="T835" device="-TO263" value="T25">
+<part name="AC/L" library="ThermoBot" deviceset="JMP-1" device="-QUICK"/>
+<part name="AC/N" library="ThermoBot" deviceset="JMP-1" device="-QUICK"/>
+<part name="JP1" library="ThermoBot" deviceset="M02" device="5MM" value="M025MM"/>
+<part name="JP3" library="ThermoBot" deviceset="M02" device="5MM" value="M025MM"/>
+<part name="U4" library="ThermoBot" deviceset="FODM3053" device=""/>
+<part name="R3" library="ThermoBot" deviceset="R-US_" device="R0805" value="100"/>
+<part name="HTR/L" library="ThermoBot" deviceset="JMP-1" device="-QUICK"/>
+<part name="HTR/N" library="ThermoBot" deviceset="JMP-1" device="-QUICK"/>
+<part name="U5" library="ThermoBot" deviceset="T835" device="-TO263" value="T25">
 <attribute name="PN-DK" value="497-10581-1-ND"/>
 </part>
-<part name="R4" library="Tempatroller" deviceset="R-US_" device="R1206" value="1k"/>
-<part name="FRAME1" library="Tempatroller" deviceset="LETTER_L" device="">
+<part name="R4" library="ThermoBot" deviceset="R-US_" device="R1206" value="1k"/>
+<part name="FRAME1" library="ThermoBot" deviceset="LETTER_L" device="">
 <attribute name="SECTION" value=""/>
 </part>
-<part name="U$1" library="Tempatroller" deviceset="SILK_QC" device="">
-<attribute name="PRODUCT" value="TempController"/>
+<part name="U$1" library="ThermoBot" deviceset="SILK_QC" device="">
+<attribute name="PRODUCT" value="ThermoBot"/>
 <attribute name="REV" value="1B"/>
 </part>
-<part name="R5" library="Tempatroller" deviceset="R-US_" device="R0805" value="390"/>
-<part name="LED1" library="Tempatroller" deviceset="LED" device="CHIP-LED0805">
+<part name="R5" library="ThermoBot" deviceset="R-US_" device="R0805" value="390"/>
+<part name="LED1" library="ThermoBot" deviceset="LED" device="CHIP-LED0805">
 <attribute name="LABEL" value="PWR"/>
 </part>
-<part name="R6" library="Tempatroller" deviceset="R-US_" device="R0805" value="390"/>
-<part name="LED2" library="Tempatroller" deviceset="LED" device="CHIP-LED0805">
+<part name="R6" library="ThermoBot" deviceset="R-US_" device="R0805" value="390"/>
+<part name="LED2" library="ThermoBot" deviceset="LED" device="CHIP-LED0805">
 <attribute name="LABEL" value="HB"/>
 </part>
-<part name="R7" library="Tempatroller" deviceset="R-US_" device="R0805" value="390"/>
-<part name="LED3" library="Tempatroller" deviceset="LED" device="CHIP-LED0805">
+<part name="R7" library="ThermoBot" deviceset="R-US_" device="R0805" value="390"/>
+<part name="LED3" library="ThermoBot" deviceset="LED" device="CHIP-LED0805">
 <attribute name="LABEL" value="SSR"/>
 </part>

Commit message: Started hardware revisions for v1B
Parts:
- removed U5: T25, ThermoBot:T835-TO263
- added JP2: M025MM, ThermoBot:M025MM
- added T1: (no value), SmslsTron:MOSFET-N-SOT23
- LED3: LABEL SSR -> TRIG
- R3: value 100 -> 10k
- R4: value 1k -> 100; device ThermoBot:R-US_R1206 -> ThermoBot:R-US_R0805
- U1: value VSK-S5 -> AC/DC-CONV-ECE05US12; device ThermoBot:VSK-S5 -> ThermoBot:AC/DC-CONV-ECE05US12
- U4: value FODM3053 -> SSR-PF240D25R; device ThermoBot:FODM3053 -> ThermoBot:SSR-PF240D25R
Connections:
- removed net N$1: R4.1, U4.A2
- removed net N$2: R3.2, U4.A
- removed net N$5: U4.A1, U5.G
- new net HTR_TRIG: JP1.1, R4.1, R7.1, T1.D1, U4.A
- net +5V: now also R3.2, R4.2
- net AC/L: now also R2.1, U4.A2; no longer R1.1, U5.A2
- net AC/L-F: no longer R4.2
- net AC/N: now also R1.1; no longer R2.1
- net GND: now also JP2.2, T1.S1
- net HTR/L: now also U4.A1; no longer U5.A1
- net HTR_SIG/D3: now also T1.G1; no longer JP1.1, R7.1
- net VIN: now also JP2.1
Other:
- note added: "Fan Output"
- moved on the sheet: HTR/L, HTR/N, JP1, LED3, R3, R4, R7, U4

Commit message: Finalized v1B design and generated MFG docs
Parts:
- U1: PN-DK 102-2387-ND -> (none)
Changed lines of the file:
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@@
 <grid distance="0.1" unitdist="inch" unit="inch" style="lines" multiple="1" display="no" altdistance="0.01" altunitdist="inch" altunit="inch"/>
 <layers>
-<layer number="1" name="Top" color="4" fill="1" visible="yes" active="no"/>
-<layer number="2" name="Route2" color="1" fill="3" visible="yes" active="no"/>
-<layer number="3" name="Route3" color="4" fill="3" visible="yes" active="no"/>
-<layer number="4" name="Route4" color="1" fill="4" visible="yes" active="no"/>
-<layer number="5" name="Route5" color="4" fill="4" visible="yes" active="no"/>
-<layer number="6" name="Route6" color="1" fill="8" visible="yes" active="no"/>
-<layer number="7" name="Route7" color="4" fill="8" visible="yes" active="no"/>
-<layer number="8" name="Route8" color="1" fill="2" visible="yes" active="no"/>
-<layer number="9" name="Route9" color="4" fill="2" visible="yes" active="no"/>
-<layer number="10" name="Route10" color="1" fill="7" visible="yes" active="no"/>
-<layer number="11" name="Route11" color="4" fill="7" visible="yes" active="no"/>
-<layer number="12" name="Route12" color="1" fill="5" visible="yes" active="no"/>
-<layer number="13" name="Route13" color="4" fill="5" visible="yes" active="no"/>
-<layer number="14" name="Route14" color="1" fill="6" visible="yes" active="no"/>
-<layer number="15" name="Route15" color="4" fill="6" visible="yes" active="no"/>
-<layer number="16" name="Bottom" color="1" fill="1" visible="yes" active="no"/>
-<layer number="17" name="Pads" color="2" fill="1" visible="yes" active="no"/>
-<layer number="18" name="Vias" color="2" fill="1" visible="yes" active="no"/>
-<layer number="19" name="Unrouted" color="6" fill="1" visible="yes" active="no"/>
-<layer number="20" name="Dimension" color="15" fill="1" visible="yes" active="no"/>
-<layer number="21" name="tPlace" color="7" fill="1" visible="yes" active="no"/>
-<layer number="22" name="bPlace" color="7" fill="1" visible="yes" active="no"/>
-<layer number="23" name="tOrigins" color="15" fill="1" visible="yes" active="no"/>
-<layer number="24" name="bOrigins" color="15" fill="1" visible="yes" active="no"/>
-<layer number="25" name="tNames" color="7" fill="1" visible="yes" active="no"/>
-<layer number="26" name="bNames" color="7" fill="1" visible="yes" active="no"/>
-<layer number="27" name="tValues" color="7" fill="1" visible="yes" active="no"/>
-<layer number="28" name="bValues" color="7" fill="1" visible="yes" active="no"/>
+<layer number="1" name="Top" color="4" fill="1" visible="no" active="no"/>
+<layer number="2" name="Route2" color="1" fill="3" visible="no" active="no"/>
+<layer number="3" name="Route3" color="4" fill="3" visible="no" active="no"/>
+<layer number="4" name="Route4" color="1" fill="4" visible="no" active="no"/>
+<layer number="5" name="Route5" color="4" fill="4" visible="no" active="no"/>
+<layer number="6" name="Route6" color="1" fill="8" visible="no" active="no"/>
+<layer number="7" name="Route7" color="4" fill="8" visible="no" active="no"/>
+<layer number="8" name="Route8" color="1" fill="2" visible="no" active="no"/>
+<layer number="9" name="Route9" color="4" fill="2" visible="no" active="no"/>
+<layer number="10" name="Route10" color="1" fill="7" visible="no" active="no"/>
+<layer number="11" name="Route11" color="4" fill="7" visible="no" active="no"/>
+<layer number="12" name="Route12" color="1" fill="5" visible="no" active="no"/>
+<layer number="13" name="Route13" color="4" fill="5" visible="no" active="no"/>
+<layer number="14" name="Route14" color="1" fill="6" visible="no" active="no"/>
+<layer number="15" name="Route15" color="4" fill="6" visible="no" active="no"/>
+<layer number="16" name="Bottom" color="1" fill="1" visible="no" active="no"/>
+<layer number="17" name="Pads" color="2" fill="1" visible="no" active="no"/>
+<layer number="18" name="Vias" color="2" fill="1" visible="no" active="no"/>
+<layer number="19" name="Unrouted" color="6" fill="1" visible="no" active="no"/>
+<layer number="20" name="Dimension" color="15" fill="1" visible="no" active="no"/>
+<layer number="21" name="tPlace" color="7" fill="1" visible="no" active="no"/>
+<layer number="22" name="bPlace" color="7" fill="1" visible="no" active="no"/>
+<layer number="23" name="tOrigins" color="15" fill="1" visible="no" active="no"/>
+<layer number="24" name="bOrigins" color="15" fill="1" visible="no" active="no"/>
+<layer number="25" name="tNames" color="7" fill="1" visible="no" active="no"/>
+<layer number="26" name="bNames" color="7" fill="1" visible="no" active="no"/>
+<layer number="27" name="tValues" color="7" fill="1" visible="no" active="no"/>
+<layer number="28" name="bValues" color="7" fill="1" visible="no" active="no"/>
 <layer number="29" name="tStop" color="2" fill="3" visible="no" active="no"/>
 <layer number="30" name="bStop" color="5" fill="6" visible="no" active="no"/>
@@
 <layer number="35" name="tGlue" color="7" fill="4" visible="no" active="no"/>
 <layer number="36" name="bGlue" color="7" fill="5" visible="no" active="no"/>
-<layer number="37" name="tTest" color="7" fill="1" visible="yes" active="no"/>
-<layer number="38" name="bTest" color="7" fill="1" visible="yes" active="no"/>
+<layer number="37" name="tTest" color="7" fill="1" visible="no" active="no"/>
+<layer number="38" name="bTest" color="7" fill="1" visible="no" active="no"/>
 <layer number="39" name="tKeepout" color="4" fill="11" visible="no" active="no"/>
 <layer number="40" name="bKeepout" color="1" fill="11" visible="no" active="no"/>
@@
 <layer number="44" name="Drills" color="7" fill="1" visible="no" active="no"/>
 <layer number="45" name="Holes" color="7" fill="1" visible="no" active="no"/>
-<layer number="46" name="Milling" color="3" fill="1" visible="yes" active="no"/>
-<layer number="47" name="Measures" color="12" fill="1" visible="yes" active="no"/>
-<layer number="48" name="Document" color="7" fill="1" visible="yes" active="no"/>
-<layer number="49" name="Reference" color="7" fill="1" visible="yes" active="no"/>
-<layer number="50" name="dxf" color="7" fill="1" visible="yes" active="no"/>
-<layer number="51" name="tDocu" color="7" fill="1" visible="yes" active="no"/>
-<layer number="52" name="bDocu" color="7" fill="1" visible="yes" active="no"/>
-<layer number="53" name="tGND_GNDA" color="7" fill="1" visible="yes" active="no"/>
-<layer number="54" name="bGND_GNDA" color="7" fill="1" visible="yes" active="no"/>
-<layer number="56" name="wert" color="7" fill="1" visible="yes" active="no"/>
-<layer number="57" name="tCAD" color="7" fill="1" visible="yes" active="no"/>
+<layer number="46" name="Milling" color="3" fill="1" visible="no" active="no"/>
+<layer number="47" name="Measures" color="12" fill="1" visible="no" active="no"/>
+<layer number="48" name="Document" color="7" fill="1" visible="no" active="no"/>
+<layer number="49" name="Reference" color="7" fill="1" visible="no" active="no"/>
+<layer number="50" name="dxf" color="7" fill="1" visible="no" active="no"/>
+<layer number="51" name="tDocu" color="7" fill="1" visible="no" active="no"/>
+<layer number="52" name="bDocu" color="7" fill="1" visible="no" active="no"/>
+<layer number="53" name="tGND_GNDA" color="7" fill="1" visible="no" active="no"/>
+<layer number="54" name="bGND_GNDA" color="7" fill="1" visible="no" active="no"/>
+<layer number="56" name="wert" color="7" fill="1" visible="no" active="no"/>
+<layer number="57" name="tCAD" color="7" fill="1" visible="no" active="no"/>
 <layer number="90" name="Modules" color="5" fill="1" visible="yes" active="yes"/>
 <layer number="91" name="Nets" color="2" fill="1" visible="yes" active="yes"/>
@@
 </class>
 <class number="1" name="MAINS-LC" width="0.508" drill="0.381">
-<clearance class="1" value="2.032"/>
+<clearance class="1" value="2.159"/>
 </class>
 <class number="2" name="MAINS-HC" width="1.27" drill="0.508">
-<clearance class="2" value="2.032"/>
+<clearance class="2" value="2.159"/>
 </class>
 </classes>
@@
 <part name="DIO-H" library="ThermoBot" deviceset="PINHD-1X10" device="TH" value="10x1F-H8.5"/>
 <part name="AIO" library="ThermoBot" deviceset="PINHD-1X6" device="TH" value="6x1F-H8.5"/>
-<part name="U1" library="ThermoBot" deviceset="AC/DC-CONV" device="-ECE05US12">
-<attribute name="PN-DK" value="102-2387-ND"/>
-</part>
+<part name="U1" library="ThermoBot" deviceset="AC/DC-CONV" device="-ECE05US12"/>
 <part name="POWER" library="ThermoBot" deviceset="PINHD-1X8" device="TH" value="8x1F-H8.5"/>
 <part name="C1" library="ThermoBot" deviceset="CPOL-US" device="153CLV-1014" value="220u">
@@
 </schematic>
 </drawing>
-<compatibility>
-<note version="6.3" minversion="6.2.2" severity="warning">
-Since Version 6.2.2 text objects can contain more than one line,
-which will not be processed correctly with this version.
-</note>
-</compatibility>
 </eagle>
